File: aux-boards/usb-socket/usb-socket.kicad_pcb (KiCad board)
At the start: 4 copper layers, 29.6 x 32.6 mm, 2 parts, among them J1 USB4056-03-A_REVA2, J5 Conn_02x12_Odd_Even

Commit message: run autoroute
Routing:
- net USB_D4: track 0.00 -> 34.5 mm
- net USB_D3: track 0.00 -> 33.0 mm
- net USB_D2: track 0.00 -> 30.5 mm
- net USB_TARGET_CC2: track 0.00 -> 29.1 mm
- net USB_D9: track 0.00 -> 28.5 mm
- net USB_D5: track 0.00 -> 23.7 mm
- net USB_D0: track 0.00 -> 19.8 mm, vias 0 -> 1
- net USB_D7: track 0.00 -> 18.6 mm
- net USB_D6: track 0.00 -> 17.8 mm
- net USB_D1: track 0.00 -> 17.7 mm
- net USB_D8: track 0.00 -> 16.1 mm
- net USB_TARGET_CC1: track 0.00 -> 16.0 mm
- net GND: track 0.00 -> 5.96 mm
- net TARGET_USB_VBUS: track 0.00 -> 2.46 mm
