File: aux-boards/breakout-board/breakout-board.kicad_pcb (KiCad board)
At the start: 4 copper layers, 52 x 38.7 mm, 28 parts, among them J1 Conn_02x06_Odd_Even, J2 USB_A, J3 Conn_ARM_SWD_TagConnect_TC2030, J5 Conn_02x12_Odd_Even, J6 Conn_01x04, SW1 SW_SPST, U1 STM32G071C8T6, U11 MAX811TEUS-T, U15 LM1117DT-3.3, U2 24LC00

Commit message: Finish aux boards
Parts:
- moved J3 1.64 mm to (118.2, 140.7)
Routing:
- net CC2: track 0.00 -> 47.4 mm
- net USB_D6: track 0.00 -> 46.6 mm, vias 0 -> 1
- net CC1: track 0.00 -> 41.8 mm, vias 0 -> 2
- net USB_D7: track 0.00 -> 36.8 mm
- net USB_D3: track 0.00 -> 35.9 mm, vias 0 -> 1
- net SDA: track 7.65 -> 41.7 mm, vias 1 -> 2
- net MCU_RESET: track 22.3 -> 55.5 mm
- net SWCLK: track 0.00 -> 32.9 mm, vias 0 -> 2
- net USB_D5: track 0.00 -> 32.7 mm
- net USB_D2: track 0.00 -> 31.2 mm
- net USB_D9: track 0.00 -> 28.2 mm
- net USB_D8: track 0.00 -> 27.1 mm
- net SWDIO: track 0.00 -> 26.4 mm, vias 0 -> 2
- net Net-(U1-PF2-NRST): track 3.86 -> 29.7 mm, vias 0 -> 2
- net SCL: track 8.76 -> 32.6 mm, vias 1 -> 2
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