File: main-board/usb-dap-rpi-probe.kicad_pcb (KiCad board)
At the start: 4 copper layers, 97.3 x 49.9 mm, 139 parts, among them J1 USB_C_Receptacle_USB2.0_16P, J2 USB_C_Receptacle_PowerOnly_6P, J3 Conn_01x02, J4 Conn_ARM_SWD_TagConnect_TC203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, J5 Conn_02x12_Odd_Even, J6 Conn_01x04, SW1 SW_SPST, U1 TUSB2036, U10 RP2350A, U11 MAX811TEUS-T, U12 USBLC6-2P6, U13 TPS259474LRPWR, U14 TPS259474LRPWR, U15 LM1117DT-3.3, U16 HT75xx-1-SOT89, U17 TPS259474LRPWR, U18 INA199xxDCK, U2 USBLC6-2P6, U24 TMUX154ERSW, U3 93CxxB, U4 W25Q128JVS, U5 FUSB302B10MPX, U6 FUSB302B11MPX, U7 MCP4451-xxxx-ST, U8 TPS259474LRPWR, U9 FUSB302B01MPX, Y1 Crystal_GND24, Y2 Crystal_GND24

Commit message: run autoroute
Parts:
- J6: moved to B.Cu
- moved J6 26.0 mm to (132.8, 143.5), turned to 180 degrees
Connections:
- J6 pad 1: GND -> INT_I2C_SDA
- J6 pad 2: +3.3V -> INT_I2C_SCL
- J6 pad 3: INT_I2C_SCL -> +3.3V
- J6 pad 4: INT_I2C_SDA -> GND
Routing:
- net MCU_USB_D-: track 20.9 -> 0.00 mm, vias 1 -> 0
- net MCU_USB_D+: track 20.5 -> 0.00 mm, vias 1 -> 0
- net GND: track 167.7 -> 164.4 mm
- net DC_IN_VBUS: track 58.8 -> 57.1 mm
- net +3.3V: track 22.1 -> 20.6 mm, vias 8 -> 7
- net USB_PWR_PRT_VBUS: track 48.7 -> 47.7 mm
- net HUB_EEPROM_MOSI: track 6.71 -> 5.94 mm
- net UPSTREAM_USB_VBUS: track 48.0 -> 47.4 mm
- net 3V3_ALW_ON: track 69.4 -> 68.8 mm
- net +1V1: track 39.4 -> 38.9 mm

Commit message: Finish routing
Parts:
- C101: footprint Capacitor_SMD:C_0402_1005Metric -> Capacitor_SMD:C_0805_2012Metric
- C11, C13, C4, C5, C6, C8: moved to B.Cu
- moved R2 22.4 mm to (117.0, 146.2), turned to 0 degrees
- moved U12 20.5 mm to (125.0, 158.0), turned to -90 degrees
- moved C4 6.73 mm to (143.4, 143.3), turned to -90 degrees
- moved C6 5.76 mm to (141.2, 138.1), turned to 45 degrees
- moved C13 4.66 mm to (145.4, 141.4), turned to 90 degrees
- moved C5 3.70 mm to (146.2, 144.3)
- moved C8 3.19 mm to (138.2, 140.4), turned to 90 degrees
- moved C11 2.98 mm to (136.2, 140.3), turned to 90 degrees
- moved C101 2.67 mm to (125.7, 132.4), turned to 180 degrees
- moved U24 2.50 mm to (126.7, 135.5)
- moved J6 2.45 mm to (130.3, 143.5)
- moved L2 2.34 mm to (132.0, 150.8)
- moved C19 2.34 mm to (132.0, 147.1)
- moved C76 1.26 mm to (91.2, 160.9), turned to -90 degrees
- moved H3 0.35 mm to (85.5, 162.2)
Routing:
- net INT_I2C_SCL: track 0.00 -> 120.9 mm, vias 0 -> 7
- net INT_I2C_SDA: track 0.00 -> 119.9 mm, vias 0 -> 5
- net Net-(U13-ILM): track 0.00 -> 112.5 mm, vias 0 -> 2
- net USB_UPSTREAM_SBU2: track 0.00 -> 74.2 mm, vias 0 -> 2
- net USB_UPSTREAM_SBU1: track 0.00 -> 72.2 mm, vias 0 -> 2
- net VBUS_2_EN: track 0.00 -> 70.6 mm, vias 0 -> 2
- net VBUS: track 42.3 -> 112.0 mm, vias 10 -> 12
- net USB_PD_INT: track 0.00 -> 67.7 mm, vias 0 -> 2
- net VBUS_0_EN: track 0.00 -> 57.7 mm, vias 0 -> 2
- net SWDIO: track 0.00 -> 52.6 mm, vias 0 -> 4
- net VBUS_1_EN: track 0.00 -> 52.4 mm, vias 0 -> 2
- net Net-(U10-GPIO27/ADC1): track 3.98 -> 53.8 mm, vias 0 -> 2
- net Net-(U10-GPIO28/ADC2): track 4.01 -> 53.7 mm, vias 0 -> 2
- net SWCLK: track 0.00 -> 48.2 mm, vias 0 -> 4
- net Net-(U10-GPIO26/ADC0): track 4.01 -> 49.3 mm
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